File: CURSED PCB/power.kicad_sch (KiCad schematic)
At the start: 22 parts, among them J3 2 Wire Block for laser, J5 G125-MH104M4-04AD000P, U1 MIC94090YC6, U2 INA180, U4 SPX3819M5-L-3-3, U5 MCP1754S-3302xCB

Commit message: Fixes to pranav sugestions
Parts:
- R6: value 198m -> 55m
Other:
- note added: "100 Gain"
- note added: "Laser: https://www.iadiy.com/infrared-laser-module-LM9IR830H200D&path=168_173"
Changed lines of the file:
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@@
 	(generator_version "9.0")
 	(paper "A4")
-	(junction
-		(at 90.17 57.15)
-		(diameter 0)
-		(color 0 0 0 0)
+	(text "100 Gain\n"
+		(exclude_from_sim no)
+		(at 103.886 78.232 0)
+		(effects
+			(font
+				(size 1.27 1.27)
+			)
+		)
+	)
+	(text "Laser: https://www.iadiy.com/infrared-laser-module-LM9IR830H200D&path=168_173"
+		(exclude_from_sim no)
+		(at 58.928 132.842 0)
+		(effects
+			(font
+				(size 1.27 1.27)
+			)
+		)
 	)
 	(junction
@@
 	)
 	(junction
+		(at 88.9 57.15)
+		(diameter 0)
+		(color 0 0 0 0)
+	)
+	(junction
 		(at 173.99 54.61)
 		(diameter 0)
@@
 	(wire
 		(pts
-			(xy 87.63 57.15) (xy 90.17 57.15)
+			(xy 87.63 57.15) (xy 88.9 57.15)
 		)
 		(stroke
@@
 	(wire
 		(pts
-			(xy 90.17 45.72) (xy 90.17 57.15)
+			(xy 88.9 45.72) (xy 88.9 57.15)
 		)
 		(stroke
@@
 	(wire
 		(pts
-			(xy 90.17 57.15) (xy 99.06 57.15)
+			(xy 88.9 57.15) (xy 99.06 57.15)
 		)
 		(stroke
@@
 	(wire
 		(pts
-			(xy 91.44 59.69) (xy 90.17 59.69)
+			(xy 78.74 72.39) (xy 90.17 72.39)
 		)
 		(stroke
@@
 	(wire
 		(pts
-			(xy 88.9 74.93) (xy 91.44 74.93)
-		)
-		(stroke
-			(width 0)
-			(type default)
-		)
-	)
-	(wire
-		(pts
 			(xy 29.21 109.22) (xy 39.37 109.22)
 		)
@@
 	(wire
 		(pts
+			(xy 88.9 57.15) (xy 88.9 77.47)
+		)
+		(stroke
+			(width 0)
+			(type default)
+		)
+	)
+	(wire
+		(pts
 			(xy 46.99 116.84) (xy 46.99 120.65)
 		)
@@
 	(wire
 		(pts
-			(xy 91.44 74.93) (xy 91.44 59.69)
-		)
-		(stroke
-			(width 0)
-			(type default)
-		)
-	)
-	(wire
-		(pts
 			(xy 45.72 86.36) (xy 54.61 86.36)
 		)
@@
 	(wire
 		(pts
-			(xy 78.74 72.39) (xy 90.17 72.39)
-		)
-		(stroke
-			(width 0)
-			(type default)
-		)
-	)
-	(wire
-		(pts
 			(xy 29.21 57.15) (xy 49.53 57.15)
 		)
@@
 	(wire
 		(pts
-			(xy 90.17 59.69) (xy 90.17 57.15)
-		)
-		(stroke
-			(width 0)
-			(type default)
-		)
-	)
-	(wire
-		(pts
 			(xy 99.06 57.15) (xy 153.67 57.15)
-		)
-		(stroke
-			(width 0)
-			(type default)
-		)
-	)
-	(wire
-		(pts
-			(xy 88.9 77.47) (xy 88.9 74.93)
 		)
 		(stroke
@@
 	(symbol
 		(lib_id "power:+3.3VA")
-		(at 90.17 45.72 0)
+		(at 88.9 45.72 0)
 		(unit 1)
 		(exclude_from_sim no)
@@
 		(fields_autoplaced yes)
 		(property "Reference" "#PWR022"
-			(at 90.17 49.53 0)
+			(at 88.9 49.53 0)
 			(effects
 				(font
@@
 		)
 		(property "Value" "+5V"
-			(at 90.17 40.64 0)
+			(at 88.9 40.64 0)
 			(effects
 				(font
@@
 		)
 		(property "Footprint" ""
-			(at 90.17 45.72 0)
+			(at 88.9 45.72 0)
 			(effects
 				(font
@@
 		)
 		(property "Datasheet" ""
-			(at 90.17 45.72 0)
+			(at 88.9 45.72 0)
 			(effects
 				(font
@@
 		)
 		(property "Description" "Power symbol creates a global label with name \"+3.3VA\""
-			(at 90.17 45.72 0)
+			(at 88.9 45.72 0)
 			(effects
 				(font
@@
 			)
 		)
-		(property "Value" "198m"
+		(property "Value" "55m"
 			(at 83.82 53.34 90)
 			(effects
