File: CURSED PCB/MCU.kicad_sch (KiCad schematic)
At the start: 22 parts, among them U1 STM32G431KBT6, U3 MIC94090YC6, Y1 24MHz crystal

Commit message: last change trust
Connections:
- net GND: no longer R15.1, U1.31 (PB8-BOOT0)
- new net: R15.1, U1.31 (PB8-BOOT0)
Changed lines of the file:
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@@
-		(color 0 0 0 0)
-	)
-	(junction
-		(at 175.26 77.47)
-		(diameter 0)
 		(color 0 0 0 0)
 	)
@@
 	(wire
 		(pts
-			(xy 175.26 77.47) (xy 185.42 77.47)
-		)
-		(stroke
-			(width 0)
-			(type default)
-		)
-	)
-	(wire
-		(pts
 			(xy 77.47 74.93) (xy 85.09 74.93)
 		)
@@
 		(pts
 			(xy 96.52 77.47) (xy 109.22 77.47)
-		)
-		(stroke
-			(width 0)
-			(type default)
-		)
-	)
-	(wire
-		(pts
-			(xy 185.42 77.47) (xy 185.42 81.28)
 		)
 		(stroke
@@
 					(unit 1)
 				)
-			)
-		)
-	)
-	(symbol
-		(lib_id "power:GND")
-		(at 185.42 81.28 0)
-		(unit 1)
-		(exclude_from_sim no)
-		(in_bom yes)
-		(on_board yes)
-		(dnp no)
-		(property "Reference" "#PWR069"
-			(at 185.42 87.63 0)
-			(effects
-				(font
-					(size 1.27 1.27)
-				)
-				(hide yes)
-			)
-		)
-		(property "Value" "GND"
-			(at 185.4201 85.09 90)
-			(effects
-				(font
-					(size 1.27 1.27)
-				)
-				(justify right)
-			)
-		)
-		(property "Footprint" ""
-			(at 185.42 81.28 0)
-			(effects
-				(font
-					(size 1.27 1.27)
-				)
-				(hide yes)
-			)
-		)
-		(property "Datasheet" ""
-			(at 185.42 81.28 0)
-			(effects
-				(font
-					(size 1.27 1.27)
-				)
-				(hide yes)
-			)
-		)
-		(property "Description" "Power symbol creates a global label with name \"GND\" , ground"
-			(at 185.42 81.28 0)
-			(effects
-				(font
-					(size 1.27 1.27)
-				)
-				(hide yes)
-			)
-		)
-		(pin "1"
-		)
-		(instances
-			(project "sensor_1"
-				(path "/9fb1a86f-679c-4b88-9ed1-932f4f414580/41420b15-6c64-4efb-bbe3-7adb1c52b946"
-					(reference "#PWR069")
-					(unit 1)
-				)
