File: CURSED PCB/PZT.kicad_sch (KiCad schematic)
At the start: 8 parts, among them U12 AD5761BRUZ

Commit message: a
Parts:
- U12: footprint AD5761BRUZ:SOP65P640X120-16N -> Package_SO:TSSOP-16_4.4x5mm_P0.65mm
Connections:
- no-connect marks 3 -> 2
Changed lines of the file:
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@@
 	(text "Acceptable Voltage Flucation of +-0.5V \nLow pass introduced to force the acceptable voltage range\n\nReistior to be found experimentally \n\nProof in google sheets labbeled \"Experimental & PCB Data Setup Master\" under Photodiode Experimental Data, \nRequirments & Comparison of PZT & Comparison of PZT to Generated Current in Payload GOogle drive"
 		(exclude_from_sim no)
-		(at 69.596 140.208 0)
+		(at 72.39 139.446 0)
 		(effects
 			(font
@@
 	)
 	(no_connect
-		(at 90.17 62.23)
-	)
-	(no_connect
 		(at 72.39 62.23)
 	)
@@
 	(wire
 		(pts
-			(xy 85.09 129.54) (xy 95.25 129.54)
-		)
-		(stroke
-			(width 0)
-			(type default)
-		)
-	)
-	(wire
-		(pts
 			(xy 69.85 92.71) (xy 72.39 92.71)
 		)
@@
 		(pts
 			(xy 116.84 106.68) (xy 120.65 106.68)
+		)
+		(stroke
+			(width 0)
+			(type default)
+		)
+	)
+	(wire
+		(pts
+			(xy 85.09 129.54) (xy 160.02 129.54)
 		)
 		(stroke
@@
 	(hierarchical_label "PZT"
 		(shape input)
-		(at 95.25 129.54 0)
+		(at 160.02 129.54 0)
 		(effects
 			(font
@@
 		)
 		(property "Description" "SMD 0201 MLCC capacitor, Alternate KiCad Library"
+			(at 142.24 96.52 0)
+			(effects
+				(font
+					(size 1.27 1.27)
+				)
+				(hide yes)
+			)
+		)
+		(property "MAXIMUN_PACKAGE_HEIGHT" ""
+			(at 142.24 96.52 0)
+			(effects
+				(font
+					(size 1.27 1.27)
+				)
+				(hide yes)
+			)
+		)
+		(property "Purchase-URL" ""
 			(at 142.24 96.52 0)
 			(effects
@@
 			)
 		)
+		(property "MAXIMUN_PACKAGE_HEIGHT" ""
+			(at 147.32 96.52 0)
+			(effects
+				(font
+					(size 1.27 1.27)
+				)
+				(hide yes)
+			)
+		)
+		(property "Purchase-URL" ""
+			(at 147.32 96.52 0)
+			(effects
+				(font
+					(size 1.27 1.27)
+				)
+				(hide yes)
+			)
+		)
 		(pin "2"
 		)
@@
 			)
 		)
+		(property "MAXIMUN_PACKAGE_HEIGHT" ""
+			(at 116.84 110.49 0)
+			(effects
+				(font
+					(size 1.27 1.27)
+				)
+				(hide yes)
+			)
+		)
+		(property "Purchase-URL" ""
+			(at 116.84 110.49 0)
+			(effects
+				(font
+					(size 1.27 1.27)
+				)
+				(hide yes)
+			)
+		)
 		(pin "2"
 		)
@@
 			)
 		)
-		(property "Footprint" "AD5761BRUZ:SOP65P640X120-16N"
+		(property "Footprint" "Package_SO:TSSOP-16_4.4x5mm_P0.65mm"
 			(at 82.55 77.47 0)
 			(effects
@@
 				)
 				(justify bottom)
+				(hide yes)
+			)
+		)
+		(property "MAXIMUN_PACKAGE_HEIGHT" ""
+			(at 82.55 77.47 90)
+			(effects
+				(font
+					(size 1.27 1.27)
+				)
+				(hide yes)
+			)
+		)
+		(property "Purchase-URL" ""
+			(at 82.55 77.47 90)
+			(effects
+				(font
+					(size 1.27 1.27)
+				)
 				(hide yes)
 			)
@@
 			)
 		)
+		(property "MAXIMUN_PACKAGE_HEIGHT" ""
+			(at 81.28 109.22 90)
+			(effects
+				(font
+					(size 1.27 1.27)
+				)
+				(hide yes)
+			)
+		)
+		(property "Purchase-URL" ""
+			(at 81.28 109.22 90)
+			(effects
+				(font
+					(size 1.27 1.27)
+				)
+				(hide yes)
+			)
+		)
 		(pin "2"
 		)
@@
 			)
 		)
+		(property "MAXIMUN_PACKAGE_HEIGHT" ""
+			(at 85.09 100.33 0)
+			(effects
+				(font
+					(size 1.27 1.27)
+				)
+				(hide yes)
+			)
+		)
+		(property "Purchase-URL" ""
+			(at 85.09 100.33 0)
+			(effects
+				(font
+					(size 1.27 1.27)
+				)
+				(hide yes)
+			)
+		)
 		(pin "2"
 		)
@@
 		)
 		(property "Description" "SMD 0201 MLCC capacitor, Alternate KiCad Library"
+			(at 110.49 110.49 0)
+			(effects
+				(font
+					(size 1.27 1.27)
+				)
+				(hide yes)
+			)
+		)
+		(property "MAXIMUN_PACKAGE_HEIGHT" ""
+			(at 110.49 110.49 0)
+			(effects
+				(font
+					(size 1.27 1.27)
+				)
+				(hide yes)
+			)
+		)
+		(property "Purchase-URL" ""
 			(at 110.49 110.49 0)
 			(effects
@@
 			(effects
 				(font
+					(size 1.27 1.27)
+				)
+				(hide yes)
+			)
+		)
+		(property "MAXIMUN_PACKAGE_HEIGHT" ""
+			(at 81.28 115.57 90)
+			(effects
+				(font
+					(size 1.27 1.27)
+				)
+				(hide yes)
+			)
+		)
+		(property "Purchase-URL" ""
+			(at 81.28 115.57 90)
+			(effects
+				(font
