File: CURSED PCB/boost.kicad_sch (KiCad schematic)
At the start: 6 parts, among them U9 TLV61046ADBVR

Commit message: a
Parts:
- removed L1: 10uH, ul_NRH3010T100MN:IND_TAIYO_NRH3010_TAY, symbol Device:L
- added L1: VLS3012CX-100M-1, VLS3012CX-100M-1:IND_VLS3012CX-100M-1, symbol VLS3012CX-100M-1:VLS3012CX-100M-1
- added TP8: 4952, testpoint:KEYSTONE_4952, symbol testpoint:4952
- U9: footprint TLV61046A:SOT95P280X145-6N -> Package_TO_SOT_SMD:TSOT-23-6_HandSoldering
Connections:
- net +24V: now also TP8.TP
- net +5V: now also L1.1
- net at U9.1 (SW): now also L1.2
